Commit message: Updated launch and added macros
Added the new macros for the lasers
Added the joint state publisher gui option to launch file
Renamed launch file to display.launch per lab instructions

File: urdf/navvis.xacro (robot description, xacro)
@@ -1,4 +1,5 @@
-<!-- <?xml version="1.0"> -->
+<!-- <?xml version="1.0"> was causing an error-->
 <robot xmlns:xacro="http://www.ros.org/wiki/xacro" name="navvis">
+    <!-- base descriptions -->
     <link name="base">
         <visual>
@@ -15,5 +16,6 @@
         </collision>
     </link>
-    <link name="laser_vert_bottom">
+    <!-- previous laser links -->
+    <!-- <link name="laser_vert_bottom">
         <visual>
             <origin xyz="0.0 0.0 0.0435" rpy="0.0 0.0 0.0"/>
@@ -29,9 +31,4 @@
         </collision>
     </link>
-    <joint name="base_laser_vert_bottom_joint " type="fixed">
-        <origin xyz="0.3158 -0.0021 0.5100" rpy="3.1355 -1.3045 0.0025"/>
-        <parent link="base"/>
-        <child link="laser_vert_bottom"/>
-    </joint>
     <link name="laser_vert_top_right">
         <visual>
@@ -48,9 +45,4 @@
         </collision>
     </link>
-    <joint name="base_laser_vert_top_right_joint " type="fixed">
-        <origin xyz="0.2978 -0.1450 1.8541" rpy="-1.1760 0.6313 -1.9377"/>
-        <parent link="base"/>
-        <child link="laser_vert_top_right"/>
-    </joint>
     <link name="laser_vert_top_left">
         <visual>
@@ -67,9 +59,4 @@
         </collision>
     </link>
-    <joint name="base_laser_vert_top_left_joint " type="fixed">
-        <origin xyz="0.2997 0.1531 1.8443" rpy="1.1780 0.6198 1.9560"/>
-        <parent link="base"/>
-        <child link="laser_vert_top_left"/>
-    </joint>
     <link name="laser_horiz">
         <visual>
@@ -85,10 +72,27 @@
             </geometry>
         </collision>
-    </link>
+    </link> -->
+    <!-- previous laser joints -->
+    <!-- <joint name="base_laser_vert_bottom_joint " type="fixed">
+        <origin xyz="0.3158 -0.0021 0.5100" rpy="3.1355 -1.3045 0.0025"/>
+        <parent link="base"/>
+        <child link="laser_vert_bottom"/>
+    </joint>
+    <joint name="base_laser_vert_top_right_joint " type="fixed">
+        <origin xyz="0.2978 -0.1450 1.8541" rpy="-1.1760 0.6313 -1.9377"/>
+        <parent link="base"/>
+        <child link="laser_vert_top_right"/>
+    </joint>
+    <joint name="base_laser_vert_top_left_joint " type="fixed">
+        <origin xyz="0.2997 0.1531 1.8443" rpy="1.1780 0.6198 1.9560"/>
+        <parent link="base"/>
+        <child link="laser_vert_top_left"/>
+    </joint>
     <joint name="base_laser_horiz_joint " type="fixed">
         <origin xyz="0.2325 0.0001 1.9201" rpy="-0.0012 0.1146 -0.0015"/>
         <parent link="base"/>
         <child link="laser_horiz"/>
-    </joint>
+    </joint> -->
+    <!-- center wheel link and joint -->
     <link name="wheel_center">
         <visual>
@@ -135,3 +139,29 @@
     <xacro:wheel side="left" reflect="1"/>
     <xacro:wheel side="right" reflect="-1"/>
+    <!-- Include the XACRO file that defines a Hokuyo LIDAR. -->
+    <xacro:include filename = "$(find gazebo_plugins)/test/multi_robot_scenario/xacro/laser/hokuyo.xacro"/>
+    <xacro:laser name = "laser_vert_bottom"
+        parent = "base"
+        xyz = "0.3157894464801903 -0.002068548615034871 0.5099999434059285"
+        rpy = "3.1354753 -1.3045001 0.0024658"
+        meshes = "package://gazebo_plugins/test/multi_robot_scenario/meshes/laser"
+    />
+    <xacro:laser name="laser_vert_top_left"
+        parent="base"
+        xyz="0.2997 0.1531 1.8443"
+        rpy="1.780 0.6198 1.9560"
+        meshes="package://gazebo_plugins/test/multi_robot_scenario/meshes/laser"
+    />
+    <xacro:laser name="laser_vert_top_right"
+        parent="base"
+        xyz="0.2978 -0.1450 1.8451"
+        rpy="-1.1760 0.6313 -1.9377"
+        meshes="package://gazebo_plugins/test/multi_robot_scenario/meshes/laser"
+    />
+    <!-- Include the XACRO file that defines a Hokuyo LIDAR. -->
+    <xacro:include filename = "$(find velodyne_description)/urdf/VLP-16.urdf.xacro"/>
+    <!-- Invoke the macro to define the Hokuyo LIDAR. -->
+    <xacro:VLP-16 parent = "base" name = "laser_horiz" topic = "laser_horiz/packets" hz = "10" samples = "440" gpu = "false">
+        <origin xyz = "0.2325416305773505 -0.0001380069427607134 1.920122926231907" rpy = "-0.0012068 0.114646 -0.0015308"/>
+    </xacro:VLP-16 >
 </robot>

Commit message: Fixed wheel rotation
Explanation in class about origin of the link vs the joint made me realize i messed it up

File: urdf/navvis.xacro (robot description, xacro)
@@ -97,5 +97,5 @@
     <link name="wheel_center">
         <visual>
-            <origin xyz="0.0 0.05 0.0" rpy="0.0 0.0 0.0"/>
+            <origin xyz="0.0 0.0 0.0" rpy="0.0 0.0 0.0"/>
             <geometry>
                 <cylinder radius="0.15" length="0.05"/>
@@ -103,5 +103,5 @@
         </visual>
         <collision>
-            <origin xyz="0.0 0.05 0.0" rpy="0.0 0.0 0.0"/>
+            <origin xyz="0.0 0.0 0.0" rpy="0.0 0.0 0.0"/>
             <geometry>
                 <cylinder radius="0.15" length="0.05"/>
@@ -110,5 +110,5 @@
     </link>
     <joint name="base_wheel_center_joint" type="continuous">
-        <origin xyz="0.10 0.05 0.0" rpy="-1.57 0.0 0.0"/>
+        <origin xyz="0.10 0.0 -0.05" rpy="-1.57 0.0 0.0"/>
         <parent link="base"/>
         <child link="wheel_center"/>
